Commit message: fake localization wip from 21/11/2018

File: p2os_urdf/defs/pioneer3at_body.xacro (robot description, xacro)
@@ -362,4 +362,18 @@
         </gazebo>
     </xacro:macro>
+<!-- Makes Gazebo publishing a ground truth position. -->
+  <xacro:macro name="stummel_ground_truth_pose">
+    <gazebo>
+      <plugin name="p3d_controller" filename="libgazebo_ros_p3d.so">
+       <alwaysOn>true</alwaysOn>
+       <updateRate>100.0</updateRate>
+       <bodyName>base_link</bodyName>
+       <topicName>ground_truth_pose</topicName>
+       <frameName>/map</frameName>
+       <xyzOffsets>1 1 0</xyzOffsets> <!-- option to initialize odometry for fake localization-->
+       <rpyOffsets>0 0 0</rpyOffsets>
+      </plugin>
+    </gazebo>
+  </xacro:macro>
     <xacro:macro name="velodyne">
         <xacro:include filename="$(find velodyne_description)/urdf/VLP-16.urdf.xacro"/>
